Commit message: Gazebo control added

File: description/robot_core.xacro (robot description, xacro)
@@ -38,7 +38,10 @@
         </collision>
         <xacro:inertial_box mass="0.5" x="0.3" y="0.3" z="0.15">
-            <orogin xyz="0.16 0 0.075" rpy="0 0 0"/>
+            <origin xyz="0.16 0 0.075" rpy="0 0 0"/>
         </xacro:inertial_box>
     </link>
+    <gazebo reference='chassis'>
+        <material>Gazebo/White</material>
+    </gazebo>
     <!-- FRONT LEFT WHEEL LINK -->
     <joint name="fl_wheel_joint" type="continuous">
@@ -64,4 +67,7 @@
         </xacro:inertial_cylinder>
     </link>
+    <gazebo reference='fl_wheel'>
+        <material>Gazebo/Blue</material>
+    </gazebo>
     <!-- FRONT RIGHT WHEEL LINK -->
     <joint name="fr_wheel_joint" type="continuous">
@@ -87,4 +93,7 @@
         </xacro:inertial_cylinder>
     </link>
+    <gazebo reference='fr_wheel'>
+        <material>Gazebo/Blue</material>
+    </gazebo>
     <!-- REAR LEFT WHEEL LINK -->
     <joint name="rl_wheel_joint" type="continuous">
@@ -110,4 +119,7 @@
         </xacro:inertial_cylinder>
     </link>
+    <gazebo reference='rl_wheel'>
+        <material>Gazebo/Blue</material>
+    </gazebo>
     <!-- REAR RIGHT WHEEL LINK -->
     <joint name="rr_wheel_joint" type="continuous">
@@ -133,3 +145,6 @@
         </xacro:inertial_cylinder>
     </link>
+    <gazebo reference='rr_wheel'>
+        <material>Gazebo/Blue</material>
+    </gazebo>
 </robot>
